Commit message: Change the urdf file of Turtlebot Waffle
Change the URDF file of Turtlebot3 Waffle, so that the robot descrption
now has an Intel Realsense RGB-D sensor mounted.

File: turtlebot3_description/urdf/turtlebot3_waffle.urdf (robot description, URDF)
Before this commit: robot turtlebot3_waffle, 13 links, 12 joints
Links:
- removed link camera_depth_frame
- removed link camera_link
- added link realsense_depth_frame
- added link realsense_link; collision box size=0.012 0.132 0.020; visual mesh filename=package://turtlebot3_description/meshes/sensors/r200.dae
Joints:
- removed joint camera_depth_joint
- added joint realsense_depth_joint: type fixed, parent realsense_link, child realsense_depth_frame, origin xyz=0.005 0.028 0.013 rpy=-1.57 0 -1.57
- joint camera_depth_optical_joint: parent camera_depth_frame -> realsense_depth_frame
- joint camera_joint: child camera_link -> realsense_link
- joint camera_rgb_joint: origin xyz=0.005 0.018 0.013 rpy=0 0 0 -> xyz=0.005 0.018 0.013 rpy=-1.57 0 -1.57; parent camera_link -> realsense_link
